Commit message: update urdf

File: hand.urdf (robot description, URDF)
Before this commit: robot glove_hand, 19 links, 18 joints
Links:
- removed link world
- added link finger1_l0; collision cylinder length=0.065 radius=0.01; visual cylinder length=0.065 radius=0.01
- added link finger2_l0; collision cylinder length=0.065 radius=0.01; visual cylinder length=0.065 radius=0.01
- added link hand_base
- added link thumb_l0; collision cylinder length=0.040 radius=0.01; visual cylinder length=0.040 radius=0.01
- link finger1_l1: mass 0.08 -> None; geometry collision cylinder length=0.090 radius=0.01; visual cylinder length=0.090 radius=0.01
- link finger1_l2: mass 0.09 -> None; geometry collision cylinder length=0.075 radius=0.01; visual cylinder length=0.075 radius=0.01
- link finger1_l3: mass 0.08 -> None; geometry collision cylinder length=0.030 radius=0.01; visual cylinder length=0.030 radius=0.01
- link finger1_l4: mass 0.04 -> None; geometry collision cylinder length=0.010 radius=0.01; visual cylinder length=0.010 radius=0.01
- link finger1_origin: mass 0.1 -> None; geometry collision sphere radius=0.025; visual sphere radius=0.025
- link finger2_l1: mass 0.08 -> None; geometry collision cylinder length=0.090 radius=0.01; visual cylinder length=0.090 radius=0.01
- link finger2_l2: mass 0.09 -> None; geometry collision cylinder length=0.075 radius=0.01; visual cylinder length=0.075 radius=0.01
- link finger2_l3: mass 0.08 -> None; geometry collision cylinder length=0.030 radius=0.01; visual cylinder length=0.030 radius=0.01
- link finger2_l4: mass 0.04 -> None; geometry collision cylinder length=0.010 radius=0.01; visual cylinder length=0.010 radius=0.01
- link finger2_origin: mass 0.1 -> None; geometry collision sphere radius=0.025; visual sphere radius=0.025
- link thumb_l1: mass 0.05 -> None; geometry collision cylinder length=0.04 radius=0.01; visual cylinder length=0.04 radius=0.01
- link thumb_l2: mass 0.05 -> None; geometry collision cylinder length=0.015 radius=0.01; visual cylinder length=0.015 radius=0.01
- link thumb_l3: mass 0.03 -> None; geometry collision cylinder length=0.045 radius=0.01; visual cylinder length=0.045 radius=0.01
- link thumb_l4: mass 0.05 -> None; geometry collision cylinder length=0.055 radius=0.01; visual cylinder length=0.055 radius=0.01
- link thumb_l5: mass 0.06 -> None; geometry collision cylinder length=0.055 radius=0.01; visual cylinder length=0.055 radius=0.01
- link thumb_l6: mass 0.06 -> None; geometry collision cylinder length=0.040 radius=0.01; visual cylinder length=0.040 radius=0.01
- link thumb_l7: mass 0.04 -> None; geometry collision cylinder length=0.020 radius=0.01; visual cylinder length=0.020 radius=0.01
- link thumb_origin: mass 0.1 -> None; geometry collision sphere radius=0.025; visual sphere radius=0.025
Joints:
- removed joint finger1_l1_joint
- removed joint finger1_l2_joint
- removed joint finger1_l3_joint
- removed joint finger1_l4_joint
- removed joint finger2_l1_joint
- removed joint finger2_l2_joint
- removed joint finger2_l3_joint
- removed joint finger2_l4_joint
- removed joint thumb_l1_joint
- removed joint thumb_l2_joint
- removed joint thumb_l3_joint
- removed joint thumb_l4_joint
- removed joint thumb_l5_joint
- removed joint thumb_l6_joint
- removed joint thumb_l7_joint
- added joint finger1_joint0: type revolute, parent finger1_origin, child finger1_l0, origin xyz=0 0 0, axis 0 0 1, limit lower=-1.5708 upper=1.5708
- added joint finger1_joint1: type revolute, parent finger1_l0, child finger1_l1, origin xyz=0.065 0 0, axis 0 1 0, limit lower=-1.5708 upper=1.5708
- added joint finger1_joint2: type revolute, parent finger1_l1, child finger1_l2, origin xyz=0.090 0 0, axis 0 1 0, limit lower=-1.5708 upper=1.5708
- added joint finger1_joint3: type revolute, parent finger1_l2, child finger1_l3, origin xyz=0.075 0 0, axis 0 1 0, limit lower=-1.5708 upper=1.5708
- added joint finger1_joint4: type revolute, parent finger1_l3, child finger1_l4, origin xyz=0.030 0 0, axis 0 1 0, limit lower=-1.5708 upper=1.5708
- added joint finger2_joint0: type revolute, parent finger2_origin, child finger2_l0, origin xyz=0 0 0, axis 0 0 1, limit lower=-1.5708 upper=1.5708
- added joint finger2_joint1: type revolute, parent finger2_l0, child finger2_l1, origin xyz=0.065 0 0, axis 0 1 0, limit lower=-1.5708 upper=1.5708
- added joint finger2_joint2: type revolute, parent finger2_l1, child finger2_l2, origin xyz=0.090 0 0, axis 0 1 0, limit lower=-1.5708 upper=1.5708
- added joint finger2_joint3: type revolute, parent finger2_l2, child finger2_l3, origin xyz=0.075 0 0, axis 0 1 0, limit lower=-1.5708 upper=1.5708
- added joint finger2_joint4: type revolute, parent finger2_l3, child finger2_l4, origin xyz=0.030 0 0, axis 0 1 0, limit lower=-1.5708 upper=1.5708
- added joint thumb_joint0: type revolute, parent thumb_origin, child thumb_l0, origin xyz=0 0 0, axis 0 0 1, limit lower=-1.5708 upper=1.5708
- added joint thumb_joint1: type revolute, parent thumb_l0, child thumb_l1, origin xyz=0.035 0 0, axis 0 1 0, limit lower=-1.5708 upper=1.5708
- added joint thumb_joint2: type revolute, parent thumb_l1, child thumb_l2, origin xyz=0.045 0 0, axis 0 0 1, limit lower=-1.5708 upper=1.5708
- added joint thumb_joint3: type revolute, parent thumb_l2, child thumb_l3, origin xyz=0.025 0 0, axis 0 0 1, limit lower=-1.5708 upper=1.5708
- added joint thumb_joint4: type revolute, parent thumb_l3, child thumb_l4, origin xyz=0.040 0 0, axis 0 1 0, limit lower=-1.5708 upper=1.5708
- added joint thumb_joint5: type revolute, parent thumb_l4, child thumb_l5, origin xyz=0.055 0 0, axis 0 1 0, limit lower=-1.5708 upper=1.5708
- added joint thumb_joint6: type revolute, parent thumb_l5, child thumb_l6, origin xyz=0.055 0 0, axis 0 1 0, limit lower=-1.5708 upper=1.5708
- added joint thumb_joint7: type revolute, parent thumb_l6, child thumb_l7, origin xyz=0.030 0 0, axis 0 1 0, limit lower=-1.5708 upper=1.5708
- joint finger1_origin_joint: origin xyz=0 0 15 rpy=0 0 0 -> xyz=0 0 0; parent world -> hand_base
- joint finger2_origin_joint: origin xyz=20 0 15 rpy=0 0 0 -> xyz=0 -0.025 0; parent world -> hand_base
- joint thumb_origin_joint: origin xyz=0 -10 5 rpy=0 0 0 -> xyz=-0.025 0 0; parent world -> hand_base

Commit message: Work on URDF visualisation in glovefox

File: hand.urdf (robot description, URDF)
Before this commit: robot glove_hand, 22 links, 21 joints
Links:
- removed link finger1_l0
- removed link finger1_l1
- removed link finger1_l2
- removed link finger1_l3
- removed link finger1_l4
- removed link finger1_origin
- removed link finger2_l0
- removed link finger2_l1
- removed link finger2_l2
- removed link finger2_l3
- removed link finger2_l4
- removed link finger2_origin
- removed link hand_base
- removed link thumb_l0
- removed link thumb_l1
- removed link thumb_l2
- removed link thumb_l3
- removed link thumb_l4
- removed link thumb_l5
- removed link thumb_l6
- removed link thumb_l7
- removed link thumb_origin
- added link F1_base; visual sphere radius=0.003
- added link F1_link0; visual cylinder length=0.065 radius=0.004
- added link F1_link1; visual cylinder length=0.090 radius=0.004
- added link F1_link2; visual cylinder length=0.075 radius=0.004
- added link F1_link3; visual cylinder length=0.030 radius=0.004
- added link F1_link4; visual cylinder length=0.010 radius=0.004
- added link F2_base; visual sphere radius=0.003
- added link F2_link0; visual cylinder length=0.065 radius=0.004
- added link F2_link1; visual cylinder length=0.090 radius=0.004
- added link F2_link2; visual cylinder length=0.075 radius=0.004
- added link F2_link3; visual cylinder length=0.030 radius=0.004
- added link F2_link4; visual cylinder length=0.010 radius=0.004
- added link T_base; visual sphere radius=0.003
- added link T_link0; visual cylinder length=0.035 radius=0.004
- added link T_link1; visual cylinder length=0.045 radius=0.004
- added link T_link2; visual cylinder length=0.025 radius=0.004
- added link T_link3; visual cylinder length=0.040 radius=0.004
- added link T_link4; visual cylinder length=0.055 radius=0.004
- added link T_link5; visual cylinder length=0.055 radius=0.004
- added link T_link6; visual cylinder length=0.030 radius=0.004
- added link T_link7; visual cylinder length=0.020 radius=0.004
Joints:
- removed joint finger1_joint0
- removed joint finger1_joint1
- removed joint finger1_joint2
- removed joint finger1_joint3
- removed joint finger1_joint4
- removed joint finger1_origin_joint
- removed joint finger2_joint0
- removed joint finger2_joint1
- removed joint finger2_joint2
- removed joint finger2_joint3
- removed joint finger2_joint4
- removed joint finger2_origin_joint
- removed joint thumb_joint0
- removed joint thumb_joint1
- removed joint thumb_joint2
- removed joint thumb_joint3
- removed joint thumb_joint4
- removed joint thumb_joint5
- removed joint thumb_joint6
- removed joint thumb_joint7
- removed joint thumb_origin_joint
- added joint F1_joint0: type continuous, parent F1_base, child F1_link0, origin xyz=0 0 0, axis 0 0 1, limit effort=1 velocity=10
- added joint F1_joint1: type continuous, parent F1_link0, child F1_link1, origin xyz=0.065 0 0, axis 0 1 0, limit effort=1 velocity=10
- added joint F1_joint2: type continuous, parent F1_link1, child F1_link2, origin xyz=0.090 0 0, axis 0 1 0, limit effort=1 velocity=10
- added joint F1_joint3: type continuous, parent F1_link2, child F1_link3, origin xyz=0.075 0 0, axis 0 1 0, limit effort=1 velocity=10
- added joint F1_joint4: type continuous, parent F1_link3, child F1_link4, origin xyz=0.030 0 0, axis 0 1 0, limit effort=1 velocity=10
- added joint F2_joint0: type continuous, parent F2_base, child F2_link0, origin xyz=0 -0.025 0, axis 0 0 1, limit effort=1 velocity=10
- added joint F2_joint1: type continuous, parent F2_link0, child F2_link1, origin xyz=0.065 0 0, axis 0 1 0, limit effort=1 velocity=10
- added joint F2_joint2: type continuous, parent F2_link1, child F2_link2, origin xyz=0.090 0 0, axis 0 1 0, limit effort=1 velocity=10
- added joint F2_joint3: type continuous, parent F2_link2, child F2_link3, origin xyz=0.075 0 0, axis 0 1 0, limit effort=1 velocity=10
- added joint F2_joint4: type continuous, parent F2_link3, child F2_link4, origin xyz=0.030 0 0, axis 0 1 0, limit effort=1 velocity=10
- added joint T_joint0: type continuous, parent T_base, child T_link0, origin xyz=-0.025 0 0, axis 0 0 1, limit effort=1 velocity=10
- added joint T_joint1: type continuous, parent T_link0, child T_link1, origin xyz=0.035 0 0, axis 0 1 0, limit effort=1 velocity=10
- added joint T_joint2: type continuous, parent T_link1, child T_link2, origin xyz=0.045 0 0, axis 0 0 1, limit effort=1 velocity=10
- added joint T_joint3: type continuous, parent T_link2, child T_link3, origin xyz=0.025 0 0, axis 0 0 1, limit effort=1 velocity=10
- added joint T_joint4: type continuous, parent T_link3, child T_link4, origin xyz=0.040 0 0, axis 0 1 0, limit effort=1 velocity=10
- added joint T_joint5: type continuous, parent T_link4, child T_link5, origin xyz=0.055 0 0, axis 0 0 1, limit effort=1 velocity=10
- added joint T_joint6: type continuous, parent T_link5, child T_link6, origin xyz=0.055 0 0, axis 0 1 0, limit effort=1 velocity=10
- added joint T_joint7: type continuous, parent T_link6, child T_link7, origin xyz=0.030 0 0, axis 0 0 1, limit effort=1 velocity=10

Commit message: fix urdf cyl and base link errors

File: hand.urdf (robot description, URDF)
Before this commit: robot hand_model, 21 links, 18 joints
Links:
- link F1_base: geometry visual sphere radius=0.01
- link F2_base: geometry visual sphere radius=0.01
- link T_base: geometry visual sphere radius=0.01
- link T_link6: geometry visual cylinder length=0.030 radius=0.004 rpy=0 0 0
Joints:
- added joint F2_OS: type fixed, parent F1_base, child F2_base, origin xyz=0 -0.025 0
- added joint T_OS: type fixed, parent F1_base, child T_base, origin xyz=-0.025 0 0
- joint T_joint0: origin xyz=-0.025 0 0 -> xyz=-0.025 0 0 rpy=0 0 1.571

Commit message: Make URDF move

File: hand.urdf (robot description, URDF)
Before this commit: robot hand_model, 21 links, 20 joints
Joints:
- joint F2_joint0: origin xyz=0 -0.025 0 -> xyz=0 0 0
- joint T_joint0: origin xyz=-0.025 0 0 rpy=0 0 1.571 -> xyz=-0 0 0 rpy=0 0 0

Commit message: add encoder publish for tumb and pointer encoders, fix joint 5 URDF

File: hand.urdf (robot description, URDF)
Before this commit: robot hand_model, 21 links, 20 joints
Joints:
- joint T_joint5: axis 0 0 1 -> 0 1 0
