Commit message: work on force feeback

File: ffb_enviroment.urdf (robot description, URDF)
Before this commit: robot ffb_environment, 3 links, 2 joints
Links:
- link thumb_ellipse: geometry visual sphere radius=0.04

Commit message: force feedback node demo ready for non thumb fingers

File: ffb_enviroment.urdf (robot description, URDF)
Before this commit: robot ffb_environment, 3 links, 2 joints
Links:
- removed link finger_plane
- link thumb_ellipse: geometry visual cylinder length=0.2 radius=0.04
Joints:
- removed joint finger_plane_joint
