Commit message: Work on joint publish

File: glove.urdf (robot description, URDF)
Before this commit: robot my_robot, 17 links, 16 joints
Links:
- removed link tl1_001
- removed link tl2_001
- removed link xc330
- added link f2xc330, mass 1; collision box size=26.000006 34.000004 20.000002; visual mesh filename=meshes/xc330_visual.stl
- added link tl1, mass 1; collision box size=18.212158 115.992867 12.568717; visual mesh filename=meshes/tl1_001_visual.stl
- added link tl2, mass 1; collision box size=14.144591 74.010262 12.10587; visual mesh filename=meshes/tl2_001_visual.stl
Joints:
- removed joint tl1_001_joint
- removed joint tl2_001_joint
- added joint tl1_joint: type revolute, parent Txc330, child tl1, origin xyz=0.653183 0.504234 -9.755316 rpy=0 0 0, axis 0 0 1, limit lower=-3.141593 upper=3.141593 effort=10 velocity=1
- added joint tl2_joint: type revolute, parent tl1, child tl2, origin xyz=-0.382935 -99.693802 0.991375 rpy=0 0 0, axis 0 0 1, limit lower=-3.141593 upper=3.141593 effort=10 velocity=1
- joint f2l1_joint: parent xc330 -> f2xc330
- joint tl3_joint: parent tl2_001 -> tl2
- joint xc330_joint: child xc330 -> f2xc330

Commit message: update state manager, rename joints

File: glove.urdf (robot description, URDF)
Before this commit: robot feedback_glove, 17 links, 16 joints
Joints:
- removed joint Txc330_joint
- removed joint bridge_joint
- removed joint f1l0_joint
- removed joint f1l1_joint
- removed joint f1l2_joint
- removed joint f1l3_joint
- removed joint f1xc330_joint
- removed joint f2l0_joint
- removed joint f2l1_joint
- removed joint f2l2_joint
- removed joint f2l3_joint
- removed joint tl0_joint
- removed joint tl1_joint
- removed joint tl2_joint
- removed joint tl3_joint
- removed joint xc330_joint
- added joint Txc330: type fixed, parent tl0, child Txc330, origin xyz=0.220604 -31.780266 1.792219 rpy=0 0 0
- added joint bridge: type fixed, parent base, child bridge
- added joint f1l0: type revolute, parent base, child f1l0, origin xyz=17.717194 -0.927605 20.41119 rpy=0 0 0, axis 0 0 1, limit lower=-3.141593 upper=3.141593 effort=10 velocity=1
- added joint f1l1: type revolute, parent f1xc330, child f1l1, origin xyz=-9.750091 0.504238 1.160593 rpy=0 0 0, axis 1 0 0, limit lower=-3.141593 upper=3.141593 effort=10 velocity=1
- added joint f1l2: type revolute, parent f1l1, child f1l2, origin xyz=0.989426 -99.801514 -0.898172 rpy=0 0 0, axis 1 0 0, limit lower=-3.141593 upper=3.141593 effort=10 velocity=1
- added joint f1l3: type revolute, parent f1l2, child f1l3, origin xyz=-0.267555 -59.855103 -0.097271 rpy=0 0 0, axis 1 0 0, limit lower=-3.141593 upper=3.141593 effort=10 velocity=1
- added joint f1xc330: type fixed, parent f1l0, child f1xc330, origin xyz=1.793839 -31.780258 -2.094622 rpy=0 0 0
- added joint f2l0: type revolute, parent base, child f2l0, origin xyz=-17.623764 -0.927605 19.505016 rpy=0 0 0, axis 0 0 1, limit lower=-3.141593 upper=3.141593 effort=10 velocity=1
- added joint f2l1: type revolute, parent f2xc330, child f2l1, origin xyz=9.750091 0.504238 2.614582 rpy=0 0 0, axis 1 0 0, limit lower=-3.141593 upper=3.141593 effort=10 velocity=1
- added joint f2l2: type revolute, parent f2l1, child f2l2, origin xyz=-0.989425 -100.17691 -2.149185 rpy=0 0 0, axis 1 0 0, limit lower=-3.141593 upper=3.141593 effort=10 velocity=1
- added joint f2l3: type revolute, parent f2l2, child f2l3, origin xyz=0.267555 -59.88974 -0.220499 rpy=0 0 0, axis 1 0 0, limit lower=-3.141593 upper=3.141593 effort=10 velocity=1
- added joint tl0: type revolute, parent base, child tl0, origin xyz=57.217976 83.967529 -24.119789 rpy=0 0 0, axis 1 0 0, limit lower=-3.141593 upper=3.141593 effort=10 velocity=1
- added joint tl1: type revolute, parent Txc330, child tl1, origin xyz=0.653183 0.504234 -9.755316 rpy=0 0 0, axis 0 0 1, limit lower=-3.141593 upper=3.141593 effort=10 velocity=1
- added joint tl2: type revolute, parent tl1, child tl2, origin xyz=-0.382935 -99.693802 0.991375 rpy=0 0 0, axis 0 0 1, limit lower=-3.141593 upper=3.141593 effort=10 velocity=1
- added joint tl3: type revolute, parent tl2, child tl3, origin xyz=-0.062885 -59.897427 0.053812 rpy=0 0 0, axis 0 0 1, limit lower=-3.141593 upper=3.141593 effort=10 velocity=1
- added joint xc330: type fixed, parent f2l0, child f2xc330, origin xyz=-1.793839 -31.780258 -1.680552 rpy=0 0 0
