Commit message: Create Gazebo bridge topic

File: glove_description/urdf/gloveold.urdf (robot description, URDF)
Before this commit: robot feedback_glove, 17 links, 16 joints
Links:
- link Txc330: mass 1e-06 -> 1; geometry collision box size=20.183695 34.000015 26.141058; visual mesh filename=package://glove_description/meshes/Txc330_visual.stl
- link base: mass 1e-06 -> 1; geometry collision box size=118.08609 200 41.493954; visual mesh filename=package://glove_description/meshes/base_visual.stl
- link bridge: mass 1e-06 -> 1; geometry collision box size=72.021408 20 38.5; visual mesh filename=package://glove_description/meshes/bridge_visual.stl
- link f1l0: mass 1e-06 -> 1; geometry collision box size=38.596191 42.810646 24.533583; visual mesh filename=package://glove_description/meshes/f1l0_visual.stl
- link f1l1: mass 1e-06 -> 1; geometry collision box size=12.441303 116.116333 18.942066; visual mesh filename=package://glove_description/meshes/f1l1_visual.stl
- link f1l2: mass 1e-06 -> 1; geometry collision box size=12.000027 74.07753 14.415758; visual mesh filename=package://glove_description/meshes/f1l2_visual.stl
- link f1l3: mass 1e-06 -> 1; geometry collision box size=25.454088 39.777729 30.544603; visual mesh filename=package://glove_description/meshes/f1l3_visual.stl
- link f1xc330: mass 1e-06 -> 1; geometry collision box size=26.000019 34.000011 20.000008; visual mesh filename=package://glove_description/meshes/f1xc330_visual.stl
- link f2l0: mass 1e-06 -> 1; geometry collision box size=38.596191 42.810646 24.533583; visual mesh filename=package://glove_description/meshes/f2l0_visual.stl
- link f2l1: mass 1e-06 -> 1; geometry collision box size=12.441278 115.97702 18.022671; visual mesh filename=package://glove_description/meshes/f2l1_visual.stl
- link f2l2: mass 1e-06 -> 1; geometry collision box size=12.000013 74 14.000005; visual mesh filename=package://glove_description/meshes/f2l2_visual.stl
- link f2l3: mass 1e-06 -> 1; geometry collision box size=25.454054 39.008659 29.511078; visual mesh filename=package://glove_description/meshes/f2l3_visual.stl
- link f2xc330: mass 1e-06 -> 1; geometry collision box size=26.000006 34.000004 20.000002; visual mesh filename=package://glove_description/meshes/xc330_visual.stl
- link tl0: mass 1e-06 -> 1; geometry collision box size=24.825493 42.810646 38.781082; visual mesh filename=package://glove_description/meshes/tl0_visual.stl
- link tl1: mass 1e-06 -> 1; geometry collision box size=18.212158 115.992867 12.568717; visual mesh filename=package://glove_description/meshes/tl1_001_visual.stl
- link tl2: mass 1e-06 -> 1; geometry collision box size=14.144591 74.010262 12.10587; visual mesh filename=package://glove_description/meshes/tl2_001_visual.stl
- link tl3: mass 1e-06 -> 1; geometry collision box size=36.27364 39.274078 28.458366; visual mesh filename=package://glove_description/meshes/tl3_visual.stl
Joints:
- joint Txc330_joint: origin xyz=0.00220604 -0.31780266 0.01792219 rpy=0 0 0 -> xyz=0.220604 -31.780266 1.792219 rpy=0 0 0
- joint f1l0_joint: origin xyz=0.17717194 -0.00927605 0.2041119 rpy=0 0 0 -> xyz=17.717194 -0.927605 20.41119 rpy=0 0 0
- joint f1l1_joint: origin xyz=-0.09750091 0.00504238 0.01160593 rpy=0 0 0 -> xyz=-9.750091 0.504238 1.160593 rpy=0 0 0
- joint f1l2_joint: origin xyz=0.00989426 -0.99801514 -0.00898172 rpy=0 0 0 -> xyz=0.989426 -99.801514 -0.898172 rpy=0 0 0
- joint f1l3_joint: origin xyz=-0.00267555 -0.59855103 -0.00097271 rpy=0 0 0 -> xyz=-0.267555 -59.855103 -0.097271 rpy=0 0 0
- joint f1xc330_joint: origin xyz=0.01793839 -0.31780258 -0.02094622 rpy=0 0 0 -> xyz=1.793839 -31.780258 -2.094622 rpy=0 0 0
- joint f2l0_joint: origin xyz=-0.17623764 -0.00927605 0.19505016 rpy=0 0 0 -> xyz=-17.623764 -0.927605 19.505016 rpy=0 0 0
- joint f2l1_joint: origin xyz=0.09750091 0.00504238 0.02614582 rpy=0 0 0 -> xyz=9.750091 0.504238 2.614582 rpy=0 0 0
- joint f2l2_joint: origin xyz=-0.00989425 -1.0017691 -0.02149185 rpy=0 0 0 -> xyz=-0.989425 -100.17691 -2.149185 rpy=0 0 0
- joint f2l3_joint: origin xyz=0.00267555 -0.5988974 -0.00220499 rpy=0 0 0 -> xyz=0.267555 -59.88974 -0.220499 rpy=0 0 0
- joint tl0_joint: origin xyz=0.57217976 0.83967529 -0.24119789 rpy=0 0 0 -> xyz=57.217976 83.967529 -24.119789 rpy=0 0 0
- joint tl1_joint: origin xyz=0.00653183 0.00504234 -0.09755316 rpy=0 0 0 -> xyz=0.653183 0.504234 -9.755316 rpy=0 0 0
- joint tl2_joint: origin xyz=-0.00382935 -0.99693802 0.00991375 rpy=0 0 0 -> xyz=-0.382935 -99.693802 0.991375 rpy=0 0 0
- joint tl3_joint: origin xyz=-0.00062885 -0.59897427 0.00053812 rpy=0 0 0 -> xyz=-0.062885 -59.897427 0.053812 rpy=0 0 0
- joint xc330_joint: origin xyz=-0.01793839 -0.31780258 -0.01680552 rpy=0 0 0 -> xyz=-1.793839 -31.780258 -1.680552 rpy=0 0 0
