Commit message: Make work in Gazebo

File: glove_description/urdf/glove.urdf (robot description, URDF)
Before this commit: robot feedback_glove, 17 links, 16 joints
Joints:
- removed joint Txc330
- removed joint bridge
- removed joint f1l0
- removed joint f1l1
- removed joint f1l2
- removed joint f1l3
- removed joint f1xc330
- removed joint f2l0
- removed joint f2l1
- removed joint f2l2
- removed joint f2l3
- removed joint tl0
- removed joint tl1
- removed joint tl2
- removed joint tl3
- removed joint xc330
- added joint Txc330_joint: type fixed, parent tl0, child Txc330, origin xyz=0.220604 -31.780266 1.792219 rpy=0 0 0
- added joint bridge_joint: type fixed, parent base, child bridge
- added joint f1l0_joint: type revolute, parent base, child f1l0, origin xyz=17.717194 -0.927605 20.41119 rpy=0 0 0, axis 0 0 1, limit lower=-3.141593 upper=3.141593 effort=10 velocity=1
- added joint f1l1_joint: type revolute, parent f1xc330, child f1l1, origin xyz=-9.750091 0.504238 1.160593 rpy=0 0 0, axis 1 0 0, limit lower=-3.141593 upper=3.141593 effort=10 velocity=1
- added joint f1l2_joint: type revolute, parent f1l1, child f1l2, origin xyz=0.989426 -99.801514 -0.898172 rpy=0 0 0, axis 1 0 0, limit lower=-3.141593 upper=3.141593 effort=10 velocity=1
- added joint f1l3_joint: type revolute, parent f1l2, child f1l3, origin xyz=-0.267555 -59.855103 -0.097271 rpy=0 0 0, axis 1 0 0, limit lower=-3.141593 upper=3.141593 effort=10 velocity=1
- added joint f1xc330_joint: type fixed, parent f1l0, child f1xc330, origin xyz=1.793839 -31.780258 -2.094622 rpy=0 0 0
- added joint f2l0_joint: type revolute, parent base, child f2l0, origin xyz=-17.623764 -0.927605 19.505016 rpy=0 0 0, axis 0 0 1, limit lower=-3.141593 upper=3.141593 effort=10 velocity=1
- added joint f2l1_joint: type revolute, parent f2xc330, child f2l1, origin xyz=9.750091 0.504238 2.614582 rpy=0 0 0, axis 1 0 0, limit lower=-3.141593 upper=3.141593 effort=10 velocity=1
- added joint f2l2_joint: type revolute, parent f2l1, child f2l2, origin xyz=-0.989425 -100.17691 -2.149185 rpy=0 0 0, axis 1 0 0, limit lower=-3.141593 upper=3.141593 effort=10 velocity=1
- added joint f2l3_joint: type revolute, parent f2l2, child f2l3, origin xyz=0.267555 -59.88974 -0.220499 rpy=0 0 0, axis 1 0 0, limit lower=-3.141593 upper=3.141593 effort=10 velocity=1
- added joint tl0_joint: type revolute, parent base, child tl0, origin xyz=57.217976 83.967529 -24.119789 rpy=0 0 0, axis 1 0 0, limit lower=-3.141593 upper=3.141593 effort=10 velocity=1
- added joint tl1_joint: type revolute, parent Txc330, child tl1, origin xyz=0.653183 0.504234 -9.755316 rpy=0 0 0, axis 0 0 1, limit lower=-3.141593 upper=3.141593 effort=10 velocity=1
- added joint tl2_joint: type revolute, parent tl1, child tl2, origin xyz=-0.382935 -99.693802 0.991375 rpy=0 0 0, axis 0 0 1, limit lower=-3.141593 upper=3.141593 effort=10 velocity=1
- added joint tl3_joint: type revolute, parent tl2, child tl3, origin xyz=-0.062885 -59.897427 0.053812 rpy=0 0 0, axis 0 0 1, limit lower=-3.141593 upper=3.141593 effort=10 velocity=1
- added joint xc330_joint: type fixed, parent f2l0, child f2xc330, origin xyz=-1.793839 -31.780258 -1.680552 rpy=0 0 0

Commit message: Make sim accept ros2 control perams

File: glove_description/urdf/glove.urdf (robot description, URDF)
Before this commit: robot feedback_glove, 17 links, 16 joints
Links:
- link Txc330: mass 1e-06 -> 0.1
- link base: mass 1e-06 -> 0.1
- link bridge: mass 1e-06 -> 0.1
- link f1l0: mass 1e-06 -> 0.1
- link f1l1: mass 1e-06 -> 0.1
- link f1l2: mass 1e-06 -> 0.1
- link f1l3: mass 1e-06 -> 0.1
- link f1xc330: mass 1e-06 -> 0.1
- link f2l0: mass 1e-06 -> 0.1
- link f2l1: mass 1e-06 -> 0.1
- link f2l2: mass 1e-06 -> 0.1
- link f2l3: mass 1e-06 -> 0.1
- link f2xc330: mass 1e-06 -> 0.1
- link tl0: mass 1e-06 -> 0.1
- link tl1: mass 1e-06 -> 0.1
- link tl2: mass 1e-06 -> 0.1
- link tl3: mass 1e-06 -> 0.1

Commit message: Update URDF to continuous joints

File: glove_description/urdf/glove.urdf (robot description, URDF)
Before this commit: robot feedback_glove, 17 links, 16 joints
Joints:
- joint f1l0_joint: limit lower=-3.141593 upper=3.141593 effort=10 velocity=1 -> (none); type revolute -> continuous
- joint f1l1_joint: limit lower=-3.141593 upper=3.141593 effort=10 velocity=1 -> (none); type revolute -> continuous
- joint f1l2_joint: limit lower=-3.141593 upper=3.141593 effort=10 velocity=1 -> (none); type revolute -> continuous
- joint f1l3_joint: limit lower=-3.141593 upper=3.141593 effort=10 velocity=1 -> (none); type revolute -> continuous
- joint f2l0_joint: limit lower=-3.141593 upper=3.141593 effort=10 velocity=1 -> (none); type revolute -> continuous
- joint f2l1_joint: limit lower=-3.141593 upper=3.141593 effort=10 velocity=1 -> (none); type revolute -> continuous
- joint f2l2_joint: limit lower=-3.141593 upper=3.141593 effort=10 velocity=1 -> (none); type revolute -> continuous
- joint f2l3_joint: limit lower=-3.141593 upper=3.141593 effort=10 velocity=1 -> (none); type revolute -> continuous
- joint tl0_joint: limit lower=-3.141593 upper=3.141593 effort=10 velocity=1 -> (none); type revolute -> continuous
- joint tl1_joint: limit lower=-3.141593 upper=3.141593 effort=10 velocity=1 -> (none); type revolute -> continuous
- joint tl2_joint: limit lower=-3.141593 upper=3.141593 effort=10 velocity=1 -> (none); type revolute -> continuous
- joint tl3_joint: limit lower=-3.141593 upper=3.141593 effort=10 velocity=1 -> (none); type revolute -> continuous

Commit message: attempt to stop vibrations and drift

File: glove_description/urdf/glove.urdf (robot description, URDF)
Before this commit: robot glove, 17 links, 16 joints
Links:
- link base: mass 0.1 -> 10
Joints:
- joint f1l0_joint: limit (none) -> lower=-12.121212 upper=12.121212 effort=10.0 velocity=20.0; type continuous -> revolute
- joint f1l1_joint: limit (none) -> lower=-12.121212 upper=12.121212 effort=10.0 velocity=20.0; type continuous -> revolute
- joint f1l2_joint: limit (none) -> lower=-12.121212 upper=12.121212 effort=10.0 velocity=20.0; type continuous -> revolute
- joint f1l3_joint: limit (none) -> lower=-12.121212 upper=12.121212 effort=10.0 velocity=20.0; type continuous -> revolute
- joint f2l0_joint: limit (none) -> lower=-12.121212 upper=12.121212 effort=10.0 velocity=20.0; type continuous -> revolute
- joint f2l1_joint: limit (none) -> lower=-12.121212 upper=12.121212 effort=10.0 velocity=20.0; type continuous -> revolute
- joint f2l2_joint: limit (none) -> lower=-12.121212 upper=12.121212 effort=10.0 velocity=20.0; type continuous -> revolute
- joint f2l3_joint: limit (none) -> lower=-12.121212 upper=12.121212 effort=10.0 velocity=20.0; type continuous -> revolute
- joint tl0_joint: limit (none) -> lower=-12.121212 upper=12.121212 effort=10.0 velocity=20.0; type continuous -> revolute
- joint tl1_joint: limit (none) -> lower=-12.121212 upper=12.121212 effort=10.0 velocity=20.0; type continuous -> revolute
- joint tl2_joint: limit (none) -> lower=-12.121212 upper=12.121212 effort=10.0 velocity=20.0; type continuous -> revolute
- joint tl3_joint: limit (none) -> lower=-12.121212 upper=12.121212 effort=10.0 velocity=20.0; type continuous -> revolute

Commit message: Work on contact sensors

File: glove_description/urdf/glove.urdf (robot description, URDF)
Before this commit: robot glove, 17 links, 16 joints
Links:
- link f1l3: mass 0.1 -> 1.0
- link f2l3: mass 0.1 -> 1.0
- link tl3: mass 0.1 -> 1.0
